File: CAD/V1.0.0/LED_dice_2.kicad_pcb (KiCad board)
At the start: 2 copper layers, 50 x 50 mm, 110 parts, among them K1 CR2032_HOLDER, Q1 NMOS-SOT-23-3, Q2 NMOS-SOT-23-3, Q3 NMOS-SOT-23-3, Q4 NMOS-SOT-23-3, U1 NE555, U2 CD4017B

Commit message: Updating open source files.
Parts:
- removed the ? at (94.8, 128.2)
- removed the D6 at (95.0, 132.0)
- renumbered D6 to D10, D7 to D11, D8 to D12, D10 to D13, D11 to D14, D12 to D15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
Routing:
- net G4: track 29.3 -> 26.6 mm
- net Net-(U2-Pad1): track 81.6 -> 79.7 mm, vias 9 -> 8
