File: CAD/V1.0.0/LED_dice_2.kicad_sch (KiCad schematic)
At the start: 46 parts, among them K1 CR2032_HOLDER, Q1 NMOS-SOT-23-3, Q2 NMOS-SOT-23-3, Q3 NMOS-SOT-23-3, Q4 NMOS-SOT-23-3, U1 NE555, U2 CD4017B

Commit message: Updating open source files.
Parts:
- renumbered D6 to D10, D7 to D11, D8 to D12, D10 to D13, D11 to D14, D12 to D15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
